File: hardware/outdoor_weather_bricklet.kicad_pcb (KiCad board)
At the start: 2 copper layers, 45 x 25 mm, 36 parts, among them J1 Debug, P1 CON-SENSOR2, P2 Boot, U1 XMC1XXX24, U2 MCP4018, U3 AM612, U4 DRILL, U5 DRILL, U6 DRILL, U7 DRILL

Commit message: briklet finished
Parts:
- removed C6, C7: 100nF, C0603F
- removed D2: red_inv, D1206_INV
- removed D3: green_inv, D1206_INV
- removed D4: blue_inv, D1206_INV
- removed the G*** at (84.1, 39.4)
- removed R2: 30k, R0603F
- removed R3, R4: 68, R0603F
- removed R5: 22, R0603F
- removed REF**: Fresnel_Lens_S8002, kicad-libraries:Fresnel_Lens_S8002
- removed RP2: 4k7, kicad-libraries:4X0603
- removed U3: AM612, AM612
- removed the VAL at (69.4, 35.2)
- removed the VAL at (51.0, 35.8)
- added ANT1: FT-004B, FT-004B, F.Cu at (82.9, 37.3)
- added VAL: WEEE_7mm, kicad-libraries:WEEE_7mm, B.Cu at (62.9, 27.3)
- added VAL: CE_5mm, kicad-libraries:CE_5mm, B.Cu at (62.9, 47.3)
- G***: moved to B.Cu
- U2: value MCP4018 -> RFM210LCF-S1; footprint kicad-libraries:SC70-6 -> RFM210LCF-S1
- U4, U5, U6, U7: footprint kicad-libraries:DRILL_NP -> DRILL_NP
- moved G*** 36.6 mm to (54.4, 20.8)
- moved C4 18.2 mm to (52.7, 31.2), turned to 180 degrees
- moved J1 17.6 mm to (49.0, 32.0)
- moved C5 13.1 mm to (73.1, 26.9), turned to 270 degrees
- moved C3 13.1 mm to (47.2, 28.1), turned to 180 degrees
- moved Fiducial_Mark 12.1 mm to (75.4, 21.3)
- moved U7 11.2 mm to (80.4, 22.3)
- moved U1 11.1 mm to (52.7, 34.9), turned to 180 degrees
- moved C2 11.0 mm to (47.4, 29.7), turned to 180 degrees
- moved U6 10.00 mm to (45.4, 22.3)
- moved R1 9.60 mm to (54.2, 43.3)
- moved D1 8.77 mm to (54.2, 44.7), turned to 0 degrees
- moved G*** 5.59 mm to (62.9, 37.3), turned to 180 degrees
- moved RP1 5.04 mm to (50.2, 39.2)
- moved C1 5.02 mm to (49.6, 41.6)
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Connections:
- C5 pad 2: VSENS -> VCC
- U1 pad 12: LED_BLUE -> (no net)
- U1 pad 13: LED_GREEN -> (no net)
- U1 pad 14: LED_RED -> (no net)
- U1 pad 16: (no net) -> SDN
- U1 pad 17: SCL -> (no net)
- U1 pad 19: SDA -> (no net)
- U1 pad 2: (no net) -> Net-(R1-Pad1)
- U1 pad 20: ENABLE -> (no net)
- U1 pad 21: VOUT -> (no net)
- U1 pad 6: (no net) -> DATA
- U1 pad 7: Net-(R1-Pad1) -> (no net)
- U2 pad 1: VCC -> Net-(ANT1-Pad1)
- U2 pad 3: SCL -> SDN
- U2 pad 4: SDA -> VCC
- U2 pad 5: VSENS -> DATA
- U2 pad 6: (no net) -> GND
Routing:
- net GND: track 25.6 -> 133.3 mm, vias 12 -> 110
- net SDN: track 0.00 -> 23.3 mm, vias 0 -> 2
- net Net-(ANT1-Pad1): track 0.00 -> 22.1 mm
- net DATA: track 0.00 -> 18.2 mm
- net SCL: track 16.3 -> 0.00 mm, vias 2 -> 0
- net VOUT: track 15.7 -> 0.00 mm
- net VCC: track 95.4 -> 81.0 mm, vias 0 -> 4
- net Net-(P2-Pad2): track 5.97 -> 19.6 mm
- net SDA: track 12.6 -> 0.00 mm, vias 2 -> 0
- net LED_GREEN: track 11.3 -> 0.00 mm
- net ENABLE: track 7.87 -> 0.00 mm
- net VSENS: track 7.79 -> 0.00 mm, vias 1 -> 0
- net LED_RED: track 6.27 -> 0.00 mm
- net LED_BLUE: track 5.01 -> 0.00 mm
- net S-MISO: track 2.55 -> 6.89 mm
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- added copper zone on F.Cu, net GND
Other:
- board size 45 x 25 mm -> 40 x 35 mm
- board text added: "Outdoor Weather 1.0"
- board text removed: "Motion Detector 2.0"

Commit message: remove silkscreen layers from footprints
Parts:
- ANT1: footprint FT-004B -> kicad-libraries:FT-004B
- U2: footprint RFM210LCF-S1 -> kicad-libraries:RFM210LCF-S1
Changed lines of the file:
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@@
     (links 43)
     (no_connects 0)
-    (area 42.709499 19.609499 83.090501 54.990501)
+    (area 42.044999 18.944999 282.27147 165.489573)
     (thickness 1.6002)
     (drawings 15)
@@
   )
   (setup
-    (last_trace_width 0.2)
+    (last_trace_width 0.29972)
     (user_trace_width 0.2)
     (user_trace_width 0.29972)
@@
       (xy 1.301301 2.715081) (xy 1.302426 2.714986)) (layer B.SilkS) (width 0.01))
   )
-  (module FT-004B (layer Vorderseite)
-    (at 82.9 37.3 270)
-    (fp_text reference ANT1 (at 0 2.5 270) (layer F.Fab)
-      (effects (font (size 0.3 0.3) (thickness 0.075)))
-    )
-    (fp_text value FT-004B (at 0 2 270) (layer F.Fab)
-      (effects (font (size 0.3 0.3) (thickness 0.075)))
-    )
-    (fp_line (start -0.5 8) (end -0.5 11) (layer F.SilkS) (width 0.5))
-    (fp_line (start -0.5 11) (end 0.5 11) (layer F.SilkS) (width 0.5))
-    (fp_line (start 0.5 11) (end 0.5 8) (layer F.SilkS) (width 0.5))
-    (fp_line (start 3 8) (end 4.5 8) (layer F.SilkS) (width 0.5))
-    (fp_line (start 4.5 8) (end 4.5 0) (layer F.SilkS) (width 0.5))
-    (fp_line (start 4.5 0) (end 3 0) (layer F.SilkS) (width 0.5))
-    (fp_line (start -3 0) (end -4.5 0) (layer F.SilkS) (width 0.5))
-    (fp_line (start -4.5 0) (end -4.5 8) (layer F.SilkS) (width 0.5))
-    (fp_line (start -4.5 8) (end -3 8) (layer F.SilkS) (width 0.5))
-    (fp_line (start 4 -6) (end -4 -6) (layer F.SilkS) (width 0.5))
-    (fp_line (start -4 -5) (end 4 -5) (layer F.SilkS) (width 0.5))
-    (fp_line (start 4 -4) (end -4 -4) (layer F.SilkS) (width 0.5))
-    (fp_line (start -4 -2) (end 4 -2) (layer F.SilkS) (width 0.5))
-    (fp_line (start -4 -3) (end 4 -3) (layer F.SilkS) (width 0.5))
-    (fp_line (start -4 -1) (end 4 -1) (layer F.SilkS) (width 0.5))
-    (fp_line (start -3 0) (end -3 -8) (layer F.SilkS) (width 0.5))
-    (fp_line (start -3 -8) (end 3 -8) (layer F.SilkS) (width 0.5))
-    (fp_line (start 3 -8) (end 3 0) (layer F.SilkS) (width 0.5))
-    (fp_line (start -3 0) (end -3 8) (layer F.SilkS) (width 0.5))
-    (fp_line (start -3 8) (end 3 8) (layer F.SilkS) (width 0.5))
-    (fp_line (start 3 8) (end 3 0) (layer F.SilkS) (width 0.5))
-    (fp_line (start 3 0) (end -3 0) (layer F.SilkS) (width 0.5))
-    (pad 2 smd rect (at -5 4 270) (size 4 8) (layers Vorderseite F.Paste F.Mask)
-      (net 1 GND))
-    (pad 2 smd rect (at 5 4 270) (size 4 8) (layers Vorderseite F.Paste F.Mask)
-      (net 1 GND))
-    (pad 1 smd rect (at 0 10.5 270) (size 3 5) (layers Vorderseite F.Paste F.Mask)
-      (net 15 "Net-(ANT1-Pad1)"))
-  )
-  (module RFM210LCF-S1 (layer Vorderseite)
-    (at 63.9 37.3 90)
-    (fp_text reference U2 (at 0 0.5 90) (layer F.Fab)
-      (effects (font (size 0.3 0.3) (thickness 0.075)))
-    )
-    (fp_text value RFM210LCF-S1 (at 0 -0.5 90) (layer F.Fab)
-      (effects (font (size 0.3 0.3) (thickness 0.075)))
-    )
-    (fp_line (start -16 -5.5) (end -16 5.5) (layer F.SilkS) (width 0.5))
-    (fp_line (start -16 5.5) (end 16 5.5) (layer F.SilkS) (width 0.5))
-    (fp_line (start 16 5.5) (end 16 -5.5) (layer F.SilkS) (width 0.5))
-    (fp_line (start 16 -5.5) (end -16 -5.5) (layer F.SilkS) (width 0.5))
-    (pad 6 smd rect (at 14.7 5.5 90) (size 1.8 5) (layers Vorderseite F.Paste F.Mask)
-      (net 1 GND))
-    (pad 5 smd rect (at 12.16 5.5 90) (size 1.8 5) (layers Vorderseite F.Paste F.Mask)
-      (net 16 DATA))
-    (pad 4 smd rect (at 9.62 5.5 90) (size 1.8 5) (layers Vorderseite F.Paste F.Mask)
-      (net 2 VCC))
-    (pad 3 smd rect (at 7.08 5.5 90) (size 1.8 5) (layers Vorderseite F.Paste F.Mask)
-      (net 17 SDN))
-    (pad 1 smd rect (at -14.7 5.5 90) (size 1.8 5) (layers Vorderseite F.Paste F.Mask)
-      (net 15 "Net-(ANT1-Pad1)"))
-    (pad 2 smd rect (at -12.16 5.5 90) (size 1.8 5) (layers Vorderseite F.Paste F.Mask)
-      (net 1 GND))
-    (pad "" smd rect (at -14.7 -5.5 90) (size 1.8 5) (layers Vorderseite F.Paste F.Mask))
-    (pad "" smd rect (at -12.16 -5.5 90) (size 1.8 5) (layers Vorderseite F.Paste F.Mask))
-  )
   (module DRILL_NP (layer Vorderseite)
     (at 45.4 52.3)
@@
       (xy 2.3114 -1.41732) (xy 2.3114 -1.67132) (xy 2.3114 -1.67132)) (layer B.SilkS) (width 0.00254))
   )
+  (module kicad-libraries:FT-004B (layer Vorderseite)
+    (at 82.9 37.3 270)
+    (fp_text reference ANT1 (at 0 2.5 270) (layer F.Fab)
+      (effects (font (size 0.3 0.3) (thickness 0.075)))
+    )
+    (fp_text value FT-004B (at 0 2 270) (layer F.Fab)
+      (effects (font (size 0.3 0.3) (thickness 0.075)))
+    )
+    (fp_line (start -0.5 8) (end -0.5 11) (layer F.Fab) (width 0.5))
+    (fp_line (start -0.5 11) (end 0.5 11) (layer F.Fab) (width 0.5))
+    (fp_line (start 0.5 11) (end 0.5 8) (layer F.Fab) (width 0.5))
+    (fp_line (start 3 8) (end 4.5 8) (layer F.Fab) (width 0.5))
+    (fp_line (start 4.5 8) (end 4.5 0) (layer F.Fab) (width 0.5))
+    (fp_line (start 4.5 0) (end 3 0) (layer F.Fab) (width 0.5))
+    (fp_line (start -3 0) (end -4.5 0) (layer F.Fab) (width 0.5))
+    (fp_line (start -4.5 0) (end -4.5 8) (layer F.Fab) (width 0.5))
+    (fp_line (start -4.5 8) (end -3 8) (layer F.Fab) (width 0.5))
+    (fp_line (start 4 -6) (end -4 -6) (layer F.Fab) (width 0.5))
+    (fp_line (start -4 -5) (end 4 -5) (layer F.Fab) (width 0.5))
+    (fp_line (start 4 -4) (end -4 -4) (layer F.Fab) (width 0.5))
+    (fp_line (start -4 -2) (end 4 -2) (layer F.Fab) (width 0.5))
+    (fp_line (start -4 -3) (end 4 -3) (layer F.Fab) (width 0.5))
+    (fp_line (start -4 -1) (end 4 -1) (layer F.Fab) (width 0.5))
+    (fp_line (start -3 0) (end -3 -8) (layer F.Fab) (width 0.5))
+    (fp_line (start -3 -8) (end 3 -8) (layer F.Fab) (width 0.5))
+    (fp_line (start 3 -8) (end 3 0) (layer F.Fab) (width 0.5))
+    (fp_line (start -3 0) (end -3 8) (layer F.Fab) (width 0.5))
+    (fp_line (start -3 8) (end 3 8) (layer F.Fab) (width 0.5))
+    (fp_line (start 3 8) (end 3 0) (layer F.Fab) (width 0.5))
+    (fp_line (start 3 0) (end -3 0) (layer F.Fab) (width 0.5))
+    (pad 2 smd rect (at -5 4 270) (size 4 8) (layers Vorderseite F.Paste F.Mask)
+      (net 1 GND))
+    (pad 2 smd rect (at 5 4 270) (size 4 8) (layers Vorderseite F.Paste F.Mask)
+      (net 1 GND))
+    (pad 1 smd rect (at 0 10.5 270) (size 3 5) (layers Vorderseite F.Paste F.Mask)
+      (net 15 "Net-(ANT1-Pad1)"))
+  )
+  (module kicad-libraries:RFM210LCF-S1 (layer Vorderseite)
+    (at 63.9 37.3 90)
+    (fp_text reference U2 (at 0 0.5 90) (layer F.Fab)
+      (effects (font (size 0.3 0.3) (thickness 0.075)))
+    )
+    (fp_text value RFM210LCF-S1 (at 0 -0.5 90) (layer F.Fab)
+      (effects (font (size 0.3 0.3) (thickness 0.075)))
+    )
+    (fp_line (start -16 -5.5) (end -16 5.5) (layer F.Fab) (width 0.5))
+    (fp_line (start -16 5.5) (end 16 5.5) (layer F.Fab) (width 0.5))
+    (fp_line (start 16 5.5) (end 16 -5.5) (layer F.Fab) (width 0.5))
+    (fp_line (start 16 -5.5) (end -16 -5.5) (layer F.Fab) (width 0.5))
+    (pad 6 smd rect (at 14.7 5.5 90) (size 1.8 5) (layers Vorderseite F.Paste F.Mask)
+      (net 1 GND))
+    (pad 5 smd rect (at 12.16 5.5 90) (size 1.8 5) (layers Vorderseite F.Paste F.Mask)
+      (net 16 DATA))
+    (pad 4 smd rect (at 9.62 5.5 90) (size 1.8 5) (layers Vorderseite F.Paste F.Mask)
+      (net 2 VCC))
+    (pad 3 smd rect (at 7.08 5.5 90) (size 1.8 5) (layers Vorderseite F.Paste F.Mask)
+      (net 17 SDN))
+    (pad 1 smd rect (at -14.7 5.5 90) (size 1.8 5) (layers Vorderseite F.Paste F.Mask)
+      (net 15 "Net-(ANT1-Pad1)"))
+    (pad 2 smd rect (at -12.16 5.5 90) (size 1.8 5) (layers Vorderseite F.Paste F.Mask)
+      (net 1 GND))
+    (pad "" smd rect (at -14.7 -5.5 90) (size 1.8 5) (layers Vorderseite F.Paste F.Mask))
+    (pad "" smd rect (at -12.16 -5.5 90) (size 1.8 5) (layers Vorderseite F.Paste F.Mask))
+  )
   (gr_line (start 82.9 40.3) (end 82.9 52.3) (angle 90) (layer Edge.Cuts) (width 0.381))

Commit message: add status led text
Other:
- board text added: "Status"
Changed lines of the file:
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@@
     (area 42.044999 18.944999 282.27147 165.489573)
     (thickness 1.6002)
-    (drawings 15)
+    (drawings 16)
     (tracks 369)
     (zones 0)
@@
   )
   (layers
-    (0 Vorderseite jumper hide)
+    (0 Vorderseite jumper)
     (31 Rückseite jumper hide)
     (32 B.Adhes user)
@@
     (aux_axis_origin 42.9 54.8)
     (grid_origin 42.9 54.8)
-    (visible_elements FFFFDFBF)
+    (visible_elements FFFFDFFF)
     (pcbplotparams
       (layerselection 0x00030_80000001)
@@
     (pad "" smd rect (at -12.16 -5.5 90) (size 1.8 5) (layers Vorderseite F.Paste F.Mask))
   )
+  (gr_text Status (at 54.2 46.3) (layer F.SilkS)
+    (effects (font (size 0.8 0.8) (thickness 0.15)))
+  )
   (gr_line (start 82.9 40.3) (end 82.9 52.3) (angle 90) (layer Edge.Cuts) (width 0.381))

Commit message: specify processor type
Parts:
- U1: value XMC1XXX24 -> XMC110024
Changed lines of the file:
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@@
       (effects (font (size 0.3 0.3) (thickness 0.075)))
     )
-    (fp_text value XMC1XXX24 (at 0 0.8 180) (layer F.Fab)
+    (fp_text value XMC110024 (at 0 0.8 180) (layer F.Fab)
       (effects (font (size 0.3 0.3) (thickness 0.075)))
     )

Commit message: Add 3d information (final)
Parts:
- ANT1: footprint kicad-libraries:FT-004B -> FT-004B
- Fiducial_Mark (x2): footprint Fiducial_Mark -> kicad-libraries:Fiducial_Mark
- U2: footprint kicad-libraries:RFM210LCF-S1 -> RFM210LCF-S1
Connections:
- P1 pad 1: (no net) -> Net-(P1-Pad1)
- U1 pad 11: (no net) -> Net-(U1-Pad11)
- U1 pad 12: (no net) -> Net-(U1-Pad12)
- U1 pad 13: (no net) -> Net-(U1-Pad13)
- U1 pad 14: (no net) -> Net-(U1-Pad14)
- U1 pad 17: (no net) -> Net-(U1-Pad17)
- U1 pad 18: (no net) -> Net-(U1-Pad18)
- U1 pad 19: (no net) -> Net-(U1-Pad19)
- U1 pad 20: (no net) -> Net-(U1-Pad20)
- U1 pad 21: (no net) -> Net-(U1-Pad21)
- U1 pad 3: (no net) -> Net-(U1-Pad3)
- U1 pad 5: (no net) -> Net-(U1-Pad5)
- U1 pad 7: (no net) -> Net-(U1-Pad7)
- U1 pad 8: (no net) -> Net-(U1-Pad8)

Commit message: Add new 3d model with more detailed components
Parts:
- ANT1: footprint FT-004B -> kicad-libraries:FT-004B
- U2: footprint RFM210LCF-S1 -> kicad-libraries:RFM210LCF-S1
