File: hardware/outdoor-weather.kicad_pcb (KiCad board)
At the start: 2 copper layers, 40 x 35 mm, 24 parts, among them J1 Debug, P1 CON-SENSOR2, P2 Boot, U1 XMC110024, U2 RFM210LCF-S1, U4 DRILL, U5 DRILL, U6 DRILL, U7 DRILL

Commit message: Change capacitor footprint(s) to C0402F
Parts:
- C1: footprint C0402E -> kicad-libraries:C0402F
- C2: footprint C0805 -> kicad-libraries:C0805
- C3, C4, C5: footprint C0603F -> kicad-libraries:C0603F
- D1: footprint D0603F -> kicad-libraries:D0603F
- R1: footprint R0603F -> kicad-libraries:R0603F
- U4, U5, U6, U7: footprint DRILL_NP -> kicad-libraries:DRILL_NP
